Commit message: removed gazebo dependency in urdf file

File: rsc/quadcopter/Hummingbird/urdf/hummingbird.urdf (robot description, URDF)
Before this commit: robot hummingbird, 6 links, 5 joints
Joints:
- joint hummingbird/rotor_0_joint: limit (none) -> effort=2000 velocity=838
- joint hummingbird/rotor_1_joint: limit (none) -> effort=2000 velocity=838
- joint hummingbird/rotor_2_joint: limit (none) -> effort=2000 velocity=838
- joint hummingbird/rotor_3_joint: limit (none) -> effort=2000 velocity=838
