Commit message: first commit for raisimGymTorch implementation

File: rsc/quadcopter/ITM_Quadrocopter/urdf/ITM_Quadrocopter.xacro (robot description, xacro)
@@ -6,5 +6,5 @@
 <robot name="ITM_Quadrocopter" xmlns:xacro="http://ros.org/wiki/xacro">
     <!-- Properties of the ITM_Quadrocopter -->
-    <xacro:property name="namespace" value="$(arg namespace)" />
+    <xacro:property name="namespace" value="ITM_Quadcopter" />
     <xacro:property name="rotor_velocity_slowdown_sim" value="10" />
     <xacro:property name="use_mesh_file" value="true" />
