Commit message: first raisimGymTorch implementation

File: rsc/quadcopter/ITM_Quadrocopter/urdf/ITM_Quadrocopter.urdf (robot description, URDF)
Before this commit: robot ITM_Quadrocopter, 6 links, 5 joints
Joints:
- joint ITM_Quadcopter/rotor_3_joint: limit (none) -> effort=2000 velocity=${max_rot_velocity}
